File: Hardware/Loadcells_Schematic.kicad_sch (KiCad schematic)
At the start: 21 parts, among them J1 LoadCell1, J2 LoadCell2, J3 LoadCell3, J4 LoadCell4, U1 ADS1115IDGS, U2 ADS1115IDGS

Commit message: Updates to PCB
Parts:
- removed R10, R9: 1k, symbol Device:R_US
Other:
- company: (none) -> ECE 405 -SIUE
- title: (none) -> ThorPCB2.0

Commit message: Updates to Sch
Connections:
- net VDD is gone; now on net +5V: C6.1, U1.1 (ADDR), U1.8 (VDD), U2.8 (VDD)
- net +Excitation renamed +5V
Changed lines of the file:
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@@
 	(wire
 		(pts
-			(xy 259.08 33.02) (xy 245.11 33.02)
+			(xy 252.73 33.02) (xy 245.11 33.02)
 		)
 		(stroke
@@
 		(pts
 			(xy 69.85 81.28) (xy 66.04 81.28)
+		)
+		(stroke
+			(width 0)
+			(type default)
+		)
+	)
+	(wire
+		(pts
+			(xy 252.73 31.75) (xy 252.73 33.02)
 		)
 		(stroke
@@
 		)
 	)
-	(label "+Excitation"
-		(at 259.08 33.02 180)
+	(label "+LoadCell3"
+		(at 38.1 73.66 0)
 		(fields_autoplaced yes)
 		(effects
@@
 				(size 1.27 1.27)
 			)
-			(justify right bottom)
-		)
-	)
-	(label "+LoadCell3"
-		(at 38.1 73.66 0)
+			(justify left bottom)
+		)
+	)
+	(hierarchical_label "SDA"
+		(shape bidirectional)
+		(at 163.83 22.86 90)
 		(fields_autoplaced yes)
 		(effects
@@
 				(size 1.27 1.27)
 			)
-			(justify left bottom)
-		)
-	)
-	(hierarchical_label "SDA"
-		(shape bidirectional)
-		(at 163.83 22.86 90)
+			(justify left)
+		)
+	)
+	(hierarchical_label "GND"
+		(shape input)
+		(at 177.8 91.44 180)
 		(fields_autoplaced yes)
 		(effects
@@
 				(size 1.27 1.27)
 			)
-			(justify left)
-		)
-	)
-	(hierarchical_label "GND"
-		(shape input)
-		(at 177.8 91.44 180)
+			(justify right)
+		)
+	)
+	(hierarchical_label "SCL"
+		(shape bidirectional)
+		(at 160.02 22.86 90)
 		(fields_autoplaced yes)
 		(effects
@@
 				(size 1.27 1.27)
 			)
-			(justify right)
-		)
-	)
-	(hierarchical_label "VDD"
-		(shape input)
-		(at 138.43 22.86 90)
-		(fields_autoplaced yes)
-		(effects
-			(font
-				(size 1.27 1.27)
-			)
-			(justify left)
-		)
-	)
-	(hierarchical_label "SCL"
-		(shape bidirectional)
-		(at 160.02 22.86 90)
-		(fields_autoplaced yes)
-		(effects
-			(font
-				(size 1.27 1.27)
-			)
 			(justify left)
 		)
@@
 	)
 	(symbol
+		(lib_id "power:+5V")
+		(at 138.43 22.86 0)
+		(unit 1)
+		(exclude_from_sim no)
+		(in_bom yes)
+		(on_board yes)
+		(dnp no)
+		(fields_autoplaced yes)
+		(property "Reference" "#PWR028"
+			(at 138.43 26.67 0)
+			(effects
+				(font
+					(size 1.27 1.27)
+				)
+				(hide yes)
+			)
+		)
+		(property "Value" "+5V"
+			(at 138.43 17.78 0)
+			(effects
+				(font
+					(size 1.27 1.27)
+				)
+			)
+		)
+		(property "Footprint" ""
+			(at 138.43 22.86 0)
+			(effects
+				(font
+					(size 1.27 1.27)
+				)
+				(hide yes)
+			)
+		)
+		(property "Datasheet" ""
+			(at 138.43 22.86 0)
+			(effects
+				(font
+					(size 1.27 1.27)
+				)
+				(hide yes)
+			)
+		)
+		(property "Description" "Power symbol creates a global label with name \"+5V\""
+			(at 138.43 22.86 0)
+			(effects
+				(font
+					(size 1.27 1.27)
+				)
+				(hide yes)
+			)
+		)
+		(pin "1"
+		)
+		(instances
+			(project "ThorPBC2.0"
+				(path "/c6e28913-7904-463c-99b0-d22103845470/327bdb77-75a9-4ebb-bd76-7bb66f9d417e"
+					(reference "#PWR028")
+					(unit 1)
+				)
+			)
+		)
+	)
+	(symbol
 		(lib_id "Analog_ADC:ADS1115IDGS")
 		(at 138.43 50.8 0)
@@
 					(unit 1)
 				)
+			)
+		)
+	)
+	(symbol
+		(lib_id "power:+5V")
+		(at 252.73 31.75 0)
+		(unit 1)
+		(exclude_from_sim no)
+		(in_bom yes)
+		(on_board yes)
+		(dnp no)
+		(fields_autoplaced yes)
+		(property "Reference" "#PWR029"
+			(at 252.73 35.56 0)
+			(effects
+				(font
+					(size 1.27 1.27)
+				)
+				(hide yes)
+			)
+		)
+		(property "Value" "+5V"
+			(at 252.73 26.67 0)
+			(effects
+				(font
+					(size 1.27 1.27)
+				)
+			)
+		)
+		(property "Footprint" ""
+			(at 252.73 31.75 0)
+			(effects
+				(font
+					(size 1.27 1.27)
+				)
+				(hide yes)
+			)
+		)
+		(property "Datasheet" ""
+			(at 252.73 31.75 0)
+			(effects
+				(font
+					(size 1.27 1.27)
+				)
+				(hide yes)
+			)
+		)
+		(property "Description" "Power symbol creates a global label with name \"+5V\""
+			(at 252.73 31.75 0)
+			(effects
+				(font
+					(size 1.27 1.27)
+				)
+				(hide yes)
+			)
+		)
+		(pin "1"
+		)
+		(instances
+			(project "ThorPBC2.0"
+				(path "/c6e28913-7904-463c-99b0-d22103845470/327bdb77-75a9-4ebb-bd76-7bb66f9d417e"
+					(reference "#PWR029")
+					(unit 1)
+				)

Commit message: Updates to Sch
Parts:
- added J8, J9: Conn_01x10_Socket, Connector_PinHeader_2.54mm:PinHeader_1x10_P2.54mm_Vertical, symbol Connector:Conn_01x10_Socket
Connections:
- net +5V: now also J8.1 (Pin_1), J9.1 (Pin_1)
- net GND: now also J8.2 (Pin_2), J9.2 (Pin_2)
- net SCL: now also J8.3 (Pin_3), J9.3 (Pin_3)
- net SDA: now also J8.4 (Pin_4), J9.4 (Pin_4)

Commit message: PCB Updates
Parts:
- removed C1, C2, C3, C4, C6: 100n, symbol Device:C
- removed J1: LoadCell1, symbol Connector:Conn_01x04_Pin
- removed J2: LoadCell2, symbol Connector:Conn_01x04_Pin
- removed J3: LoadCell3, symbol Connector:Conn_01x04_Pin
- removed J4: LoadCell4, symbol Connector:Conn_01x04_Pin
- removed R1, R2, R3, R4, R5, R6, R7, R8: 100, symbol Device:R_US
- added C1, C2, C3, C4, C6: 0.1uF, ThorParts:CAP_C320_KEM, symbol 2024-10-08_02-19-51:C320C104K5R5TA
- added J10, J11, J12, J13: Screw_Terminal_01x04, TerminalBlock_Phoenix:TerminalBlock_Phoenix_MPT-0,5-4-2.54_1x04_P2.54mm_Horizontal, symbol Connector:Screw_Terminal_01x04
- added R1, R2, R3, R4, R5, R6, R7, R8: 100 Ohms, RES_TYCO_YR1_TYC, symbol 2024-10-08_02-54-42:YR1B100RCC
Connections:
- net +5V: now also J9.5 (Pin_5), C6.1, J10.1 (Pin_1), J11.1 (Pin_1), J12.1 (Pin_1), J13.1 (Pin_1)
- net +LoadCell1: now also J10.4 (Pin_4), R1.1
- net +LoadCell2: now also J11.4 (Pin_4), R3.1
- net +LoadCell3: now also J12.4 (Pin_4), R5.1
- net +LoadCell4: now also J13.4 (Pin_4), R7.1
- net -LoadCell1: now also J10.3 (Pin_3), R2.1
- net -LoadCell2: now also J11.3 (Pin_3), R4.1
- net -LoadCell3: now also J12.3 (Pin_3), R6.1
- net -LoadCell4: now also J13.3 (Pin_3), R8.1
- net GND: now also J8.5 (Pin_5), C6.2, J10.2 (Pin_2), J11.2 (Pin_2), J12.2 (Pin_2), J13.2 (Pin_2)
- net 1_A3: now reaches U1.6 (AIN2)
- net 1_A3: now also J9.9 (Pin_9), C4.1, R7.2
- net 1_A1: now reaches U1.4 (AIN0)
- net 1_A1: now also J9.7 (Pin_7), C3.1, R5.2
- net 1_A2: now reaches U1.5 (AIN1)
- net 1_A2: now also J9.8 (Pin_8), C3.2, R6.2
- net 1_A4: now reaches U1.7 (AIN3)
- net 1_A4: now also J9.10 (Pin_10), C4.2, R8.2
- net 2_A1: now reaches U2.4 (AIN0)
- net 2_A1: now also J8.7 (Pin_7), C1.1, R1.2
- net 2_A2: now reaches U2.5 (AIN1)
- net 2_A2: now also J8.8 (Pin_8), C1.2, R2.2
- net 2_A3: now reaches U2.6 (AIN2)
- net 2_A3: now also J8.9 (Pin_9), C2.1, R3.2
- net 2_A4: now reaches U2.7 (AIN3)
- net 2_A4: now also J8.10 (Pin_10), C2.2, R4.2
- no-connect marks 0 -> 4

Commit message: Updates to PCB
Parts:
- J10: value Screw_Terminal_01x04 -> LoadCell_0
- J11: value Screw_Terminal_01x04 -> LoadCell_1
- J12: value Screw_Terminal_01x04 -> LoadCell_2
- J13: value Screw_Terminal_01x04 -> LoadCell_3
- J8: value Conn_01x10_Socket -> ADS1115_Module_1; footprint Connector_PinHeader_2.54mm:PinHeader_1x10_P2.54mm_Vertical -> ThorParts:ADS1115_1x10_P2.54mm_Vertical
- J9: value Conn_01x10_Socket -> ADS1115_Module_0; footprint Connector_PinHeader_2.54mm:PinHeader_1x10_P2.54mm_Vertical -> ThorParts:ADS1115_1x10_P2.54mm_Vertical
Changed lines of the file:
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@@
 			)
 		)
-		(property "Value" "Screw_Terminal_01x04"
+		(property "Value" "LoadCell_2"
 			(at 240.03 69.8499 0)
 			(effects
@@
 		(exclude_from_sim no)
 		(in_bom yes)
-		(on_board yes)
+		(on_board no)
 		(dnp no)
 		(fields_autoplaced yes)
@@
 			)
 		)
-		(property "Value" "Conn_01x10_Socket"
+		(property "Value" "ADS1115_Module_1"
 			(at 71.12 139.6999 0)
 			(effects
@@
 			)
 		)
-		(property "Footprint" "Connector_PinHeader_2.54mm:PinHeader_1x10_P2.54mm_Vertical"
+		(property "Footprint" "ThorParts:ADS1115_1x10_P2.54mm_Vertical"
 			(at 69.85 137.16 0)
 			(effects
@@
 			)
 		)
-		(property "Value" "Screw_Terminal_01x04"
+		(property "Value" "LoadCell_0"
 			(at 240.03 43.1799 0)
 			(effects
@@
 			)
 		)
-		(property "Value" "Screw_Terminal_01x04"
+		(property "Value" "LoadCell_3"
 			(at 240.03 83.8199 0)
 			(effects
@@
 			)
 		)
-		(property "Value" "Conn_01x10_Socket"
+		(property "Value" "ADS1115_Module_0"
 			(at 71.12 170.1799 0)
 			(effects
@@
 			)
 		)
-		(property "Footprint" "Connector_PinHeader_2.54mm:PinHeader_1x10_P2.54mm_Vertical"
+		(property "Footprint" "ThorParts:ADS1115_1x10_P2.54mm_Vertical"
 			(at 69.85 167.64 0)
 			(effects
@@
 			)
 		)
-		(property "Value" "Screw_Terminal_01x04"
+		(property "Value" "LoadCell_1"
 			(at 240.03 55.8799 0)
 			(effects
