File: Hardware/StepperDriver.kicad_sch (KiCad schematic)
At the start: 4 parts, among them M1 Stepper_Motor_bipolar, U3 L293D

Commit message: Updates to PCB
Other:
- company: (none) -> ECE 405 -SIUE
- title: (none) -> ThorPCB2.0
Changed lines of the file:
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@@
 	(generator "eeschema")
 	(generator_version "8.0")
-	(paper "A4")
+	(paper "USLetter")
+	(title_block
+		(title "ThorPCB2.0")
+		(company "ECE 405 -SIUE")
+	)
 	(junction
 		(at 146.05 118.11)

Commit message: Updates to Sch
Parts:
- C10: value 0.1u -> 1u
Connections:
- net VCC1 renamed +5V
- net VCC2 renamed +12V
Changed lines of the file:
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@@
+	)
+	(junction
+		(at 146.05 60.96)
+		(diameter 0)
+		(color 0 0 0 0)
 	)
 	(junction
@@
 		(color 0 0 0 0)
 	)
-	(junction
-		(at 146.05 60.96)
-		(diameter 0)
-		(color 0 0 0 0)
-	)
 	(wire
 		(pts
@@
 	(wire
 		(pts
+			(xy 146.05 60.96) (xy 152.4 60.96)
+		)
+		(stroke
+			(width 0)
+			(type default)
+		)
+	)
+	(wire
+		(pts
 			(xy 140.97 63.5) (xy 140.97 67.31)
 		)
@@
 	(wire
 		(pts
-			(xy 140.97 58.42) (xy 140.97 63.5)
+			(xy 140.97 55.88) (xy 140.97 63.5)
 		)
 		(stroke
@@
 	(wire
 		(pts
-			(xy 146.05 58.42) (xy 146.05 60.96)
-		)
-		(stroke
-			(width 0)
-			(type default)
-		)
-	)
-	(wire
-		(pts
 			(xy 101.6 64.77) (xy 101.6 63.5)
 		)
@@
 		(pts
 			(xy 146.05 118.11) (xy 148.59 118.11)
+		)
+		(stroke
+			(width 0)
+			(type default)
+		)
+	)
+	(wire
+		(pts
+			(xy 152.4 55.88) (xy 152.4 60.96)
 		)
 		(stroke
@@
 		)
 	)
-	(hierarchical_label "VCC1"
+	(hierarchical_label "1A"
 		(shape input)
-		(at 140.97 58.42 90)
+		(at 114.3 77.47 180)
 		(fields_autoplaced yes)
 		(effects
@@
 				(size 1.27 1.27)
 			)
-			(justify left)
-		)
-	)
-	(hierarchical_label "1A"
+			(justify right)
+		)
+	)
+	(hierarchical_label "4A"
 		(shape input)
-		(at 114.3 77.47 180)
+		(at 114.3 97.79 180)
 		(fields_autoplaced yes)
 		(effects
@@
 		)
 	)
-	(hierarchical_label "4A"
+	(hierarchical_label "2A"
 		(shape input)
-		(at 114.3 97.79 180)
+		(at 114.3 82.55 180)
 		(fields_autoplaced yes)
 		(effects
@@
 		)
 	)
-	(hierarchical_label "2A"
+	(hierarchical_label "3A"
 		(shape input)
-		(at 114.3 82.55 180)
+		(at 114.3 92.71 180)
 		(fields_autoplaced yes)
 		(effects
@@
 		)
 	)
-	(hierarchical_label "3A"
+	(hierarchical_label "GND"
 		(shape input)
-		(at 114.3 92.71 180)
+		(at 165.1 115.57 180)
 		(fields_autoplaced yes)
 		(effects
@@
 			)
 			(justify right)
-		)
-	)
-	(hierarchical_label "GND"
-		(shape input)
-		(at 165.1 115.57 180)
-		(fields_autoplaced yes)
-		(effects
-			(font
-				(size 1.27 1.27)
-			)
-			(justify right)
-		)
-	)
-	(hierarchical_label "VCC2"
-		(shape input)
-		(at 146.05 58.42 90)
-		(fields_autoplaced yes)
-		(effects
-			(font
-				(size 1.27 1.27)
-			)
-			(justify left)
 		)
 	)
@@
 			)
 		)
-		(property "Value" "0.1u"
+		(property "Value" "1u"
 			(at 93.98 67.3099 0)
 			(effects
@@
 	)
 	(symbol
+		(lib_id "power:+12V")
+		(at 152.4 55.88 0)
+		(unit 1)
+		(exclude_from_sim no)
+		(in_bom yes)
+		(on_board yes)
+		(dnp no)
+		(fields_autoplaced yes)
+		(property "Reference" "#PWR032"
+			(at 152.4 59.69 0)
+			(effects
+				(font
+					(size 1.27 1.27)
+				)
+				(hide yes)
+			)
+		)
+		(property "Value" "+12V"
+			(at 152.4 50.8 0)
+			(effects
+				(font
+					(size 1.27 1.27)
+				)
+			)
+		)
+		(property "Footprint" ""
+			(at 152.4 55.88 0)
+			(effects
+				(font
+					(size 1.27 1.27)
+				)
+				(hide yes)
+			)
+		)
+		(property "Datasheet" ""
+			(at 152.4 55.88 0)
+			(effects
+				(font
+					(size 1.27 1.27)
+				)
+				(hide yes)
+			)
+		)
+		(property "Description" "Power symbol creates a global label with name \"+12V\""
+			(at 152.4 55.88 0)
+			(effects
+				(font
+					(size 1.27 1.27)
+				)
+				(hide yes)
+			)
+		)
+		(pin "1"
+		)
+		(instances
+			(project "ThorPBC2.0"
+				(path "/c6e28913-7904-463c-99b0-d22103845470/931e2ded-8ee9-46d5-bece-ca163642fd90"
+					(reference "#PWR032")
+					(unit 1)
+				)
+				(path "/c6e28913-7904-463c-99b0-d22103845470/22174d40-6f09-42c0-b922-da63a0962664"
+					(reference "#PWR033")
+					(unit 1)
+				)
+				(path "/c6e28913-7904-463c-99b0-d22103845470/e4d1719b-ab9c-4829-9c6a-900123a30a32"
+					(reference "#PWR034")
+					(unit 1)
+				)
+				(path "/c6e28913-7904-463c-99b0-d22103845470/3f1e802e-a354-41d9-9508-14e9ab0b0748"
+					(reference "#PWR035")
+					(unit 1)
+				)
+			)
+		)
+	)
+	(symbol
 		(lib_id "Driver_Motor:L293D")
 		(at 143.51 92.71 0)
@@
 					(unit 1)
 				)
+			)
+		)
+	)
+	(symbol
+		(lib_id "power:+5V")
+		(at 140.97 55.88 0)
+		(unit 1)
+		(exclude_from_sim no)
+		(in_bom yes)
+		(on_board yes)
+		(dnp no)
+		(fields_autoplaced yes)
+		(property "Reference" "#PWR036"
+			(at 140.97 59.69 0)
+			(effects
+				(font
+					(size 1.27 1.27)
+				)
+				(hide yes)
+			)
+		)
+		(property "Value" "+5V"
+			(at 140.97 50.8 0)
+			(effects
+				(font
+					(size 1.27 1.27)
+				)
+			)
+		)
+		(property "Footprint" ""
+			(at 140.97 55.88 0)
+			(effects
+				(font
+					(size 1.27 1.27)
+				)
+				(hide yes)
+			)
+		)
+		(property "Datasheet" ""
+			(at 140.97 55.88 0)
+			(effects
+				(font
+					(size 1.27 1.27)
+				)
+				(hide yes)
+			)
+		)
+		(property "Description" "Power symbol creates a global label with name \"+5V\""
+			(at 140.97 55.88 0)
+			(effects
+				(font
+					(size 1.27 1.27)
+				)
+				(hide yes)
+			)
+		)
+		(pin "1"
+		)
+		(instances
+			(project "ThorPBC2.0"
+				(path "/c6e28913-7904-463c-99b0-d22103845470/931e2ded-8ee9-46d5-bece-ca163642fd90"
+					(reference "#PWR036")
+					(unit 1)
+				)
+				(path "/c6e28913-7904-463c-99b0-d22103845470/22174d40-6f09-42c0-b922-da63a0962664"
+					(reference "#PWR037")
+					(unit 1)
+				)
+				(path "/c6e28913-7904-463c-99b0-d22103845470/e4d1719b-ab9c-4829-9c6a-900123a30a32"
+					(reference "#PWR038")
+					(unit 1)
+				)
+				(path "/c6e28913-7904-463c-99b0-d22103845470/3f1e802e-a354-41d9-9508-14e9ab0b0748"
+					(reference "#PWR039")
+					(unit 1)
+				)

Commit message: PCB Updates
Parts:
- removed C10: 1u, symbol Device:C
- removed C5: 0.1u, symbol Device:C
- added C10: 1uF, ThorParts:CAP_C330C_MR_X7R_KEM, symbol 2024-10-08_03-02-35:C330C105K5R5TA7301
- added C5: 0.1uF, ThorParts:CAP_C320_KEM, symbol 2024-10-08_02-19-51:C320C104K5R5TA
- M1: footprint Connector_PinHeader_2.54mm:PinHeader_1x04_P2.54mm_Vertical -> TerminalBlock_Phoenix:TerminalBlock_Phoenix_MPT-0,5-4-2.54_1x04_P2.54mm_Horizontal
Connections:
- net +12V: now also C10.1
- net +5V: now also C5.1
- net GND: now also C10.2, C5.2

Commit message: Updates to PCB
Parts:
- M1: value Stepper_Motor_bipolar -> Stepper_Motor
Changed lines of the file:
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@@
 			)
 		)
-		(property "Value" "Stepper_Motor_bipolar"
+		(property "Value" "Stepper_Motor"
 			(at 181.61 95.669 0)
 			(effects
