File: Hardware/ThorPBC2.0.kicad_pcb (KiCad board)
At the start: 2 copper layers, 40 parts, among them J10 Screw_Terminal_01x04, J11 Screw_Terminal_01x04, J12 Screw_Terminal_01x04, J13 Screw_Terminal_01x04, J5 Conn_01x03_Pin, J6 ATX-24, J7 Conn_01x03_Pin, J8 Conn_01x10_Socket, J9 Conn_01x10_Socket, M1 Stepper_Motor_bipolar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

Commit message: Updates to PCB
Parts:
- removed C6: 0.1uF, ThorParts:CAP_C320_KEM
- moved J6 102.4 mm to (164.0, 74.1), turned to -90 degrees
- moved SW1 40.4 mm to (152.0, 65.5), turned to 90 degrees
- moved M3 35.7 mm to (118.7, 169.2)
- moved M2 34.1 mm to (96.2, 169.6)
- moved M1 31.7 mm to (70.7, 168.2)
- moved C12 26.5 mm to (115.0, 156.4), turned to -90 degrees
- moved C11 23.5 mm to (92.3, 157.2), turned to -90 degrees
- moved C8 22.8 mm to (126.9, 134.5)
- moved C10 22.1 mm to (66.5, 156.9), turned to -90 degrees
- moved C7 20.1 mm to (104.2, 135.2)
- moved C5 20.1 mm to (78.4, 135.1)
- moved J5 14.6 mm to (111.9, 97.4)
- moved U7 14.4 mm to (131.5, 96.0)
- moved J7 14.4 mm to (111.9, 71.6)
- moved C2 12.3 mm to (79.1, 86.6)
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Routing:
- net /Loadcell_ADCs/-LoadCell1: track 0.00 -> 12.6 mm
- net /Loadcell_ADCs/-LoadCell3: track 0.00 -> 12.2 mm
- net /Loadcell_ADCs/-LoadCell2: track 0.00 -> 12.2 mm
- net /Loadcell_ADCs/-LoadCell4: track 0.00 -> 12.0 mm
- added copper zone on In2.Cu, net +12V
- added copper zone on In2.Cu, net +5V
- added copper zone on In1.Cu, net GND
Other:
- board outline added: 127 x 115.5 mm
- copper layers 2 -> 4

Commit message: Updates to PCB
Parts:
- added REF**: MountingHole_2.5mm_Pad_TopBottom, MountingHole:MountingHole_2.5mm_Pad_TopBottom, F.Cu at (54.5, 168.5)
- added REF**: MountingHole_2.5mm_Pad_TopBottom, MountingHole:MountingHole_2.5mm_Pad_TopBottom, F.Cu at (167.0, 135.0)
- added REF**: MountingHole_2.5mm_Pad_TopBottom, MountingHole:MountingHole_2.5mm_Pad_TopBottom, F.Cu at (54.5, 65.5)
- added REF**: MountingHole_2.5mm_Pad_TopBottom, MountingHole:MountingHole_2.5mm_Pad_TopBottom, F.Cu at (166.5, 65.5)
- added REF**: MountingHole_2.5mm_Pad_TopBottom, MountingHole:MountingHole_2.5mm_Pad_TopBottom, F.Cu at (167.0, 169.0)
- J10: value Screw_Terminal_01x04 -> LoadCell_0
- J11: value Screw_Terminal_01x04 -> LoadCell_1
- J12: value Screw_Terminal_01x04 -> LoadCell_2
- J13: value Screw_Terminal_01x04 -> LoadCell_3
- J5: value Conn_01x03_Pin -> UART_1
- J7: value Conn_01x03_Pin -> UART_0
- J8: value Conn_01x10_Socket -> ADS1115_Module_1; footprint Connector_PinHeader_2.54mm:PinHeader_1x10_P2.54mm_Vertical -> ThorParts:ADS1115_1x10_P2.54mm_Vertical
- J9: value Conn_01x10_Socket -> ADS1115_Module_0; footprint Connector_PinHeader_2.54mm:PinHeader_1x10_P2.54mm_Vertical -> ThorParts:ADS1115_1x10_P2.54mm_Vertical
- M1, M2, M3, M4: value Stepper_Motor_bipolar -> Stepper_Motor
- moved J7 5.35 mm to (112.8, 76.9)
- moved J8 5.26 mm to (90.5, 68.1)
- moved J9 5.26 mm to (90.5, 102.5)
- moved U7 5.02 mm to (132.0, 101.0)
- moved J5 5.00 mm to (112.9, 102.3)
- moved C1 3.96 mm to (83.0, 73.8)
- moved C2 3.96 mm to (82.5, 88.5)
- moved C3 3.96 mm to (82.5, 103.6)
- moved C4 3.96 mm to (82.5, 118.7)
- moved R1 3.96 mm to (67.3, 72.8)
- moved R5 3.96 mm to (66.8, 102.8)
- moved R6 3.96 mm to (66.8, 106.9)
- moved R7 3.96 mm to (66.3, 117.8)
- moved R8 3.96 mm to (66.3, 121.9)
- moved J10 3.96 mm to (55.2, 80.4)
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Routing:
- net /SCL: track 0.00 -> 75.8 mm
- net /SDA: track 0.00 -> 73.7 mm
- net Net-(J6-PS_ON#): track 0.00 -> 25.6 mm
- net /Loadcell_ADCs/1_A1: track 4.62 -> 22.1 mm
- net /Loadcell_ADCs/1_A2: track 4.64 -> 22.1 mm
- net /Loadcell_ADCs/2_A2: track 4.59 -> 17.3 mm
- net /Loadcell_ADCs/2_A1: track 4.70 -> 17.4 mm
- net /UART0_RX: track 0.00 -> 10.3 mm
- net /UART0_TX: track 0.00 -> 10.3 mm
- net /UART1_TX: track 0.00 -> 10.2 mm
- net /UART1_RX: track 0.00 -> 10.2 mm
- net /Loadcell_ADCs/1_A3: track 5.17 -> 14.9 mm
- net /Loadcell_ADCs/1_A4: track 5.10 -> 14.8 mm
- net /Loadcell_ADCs/2_A3: track 4.66 -> 12.7 mm
- net /Loadcell_ADCs/2_A4: track 4.71 -> 12.8 mm
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Other:
- board size 127 x 115.5 mm -> 123 x 113.5 mm

Commit message: Updates to PCB
Parts:
- added G***: LOGO, ThorParts:SIUE_Logo, F.Cu at (54.0, 146.5)
- moved M3 1.08 mm to (121.0, 167.5)
- moved M2 0.62 mm to (95.5, 167.5)
- moved J13 0.50 mm to (55.5, 125.4)
- moved M4 0.50 mm to (145.5, 167.5)
- moved M1 0.12 mm to (70.5, 167.5)
Routing:
- net +5V: track 0.00 -> 81.5 mm
- net /12A: track 0.00 -> 73.7 mm
- net /42A: track 0.00 -> 72.6 mm
- net /13A: track 0.00 -> 67.1 mm
- net /11A: track 0.00 -> 65.9 mm
- net /41A: track 0.00 -> 63.5 mm
- net /43A: track 0.00 -> 57.2 mm
- net /14A: track 0.00 -> 55.2 mm
- net /24A: track 0.00 -> 51.8 mm
- net /23A: track 0.00 -> 51.4 mm
- net /32A: track 0.00 -> 51.3 mm
- net /33A: track 0.00 -> 45.7 mm
- net /22A: track 0.00 -> 42.5 mm
- net /44A: track 0.00 -> 40.3 mm
- net /31A: track 0.00 -> 38.2 mm
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Other:
- board text added: "ECE 405 Senior Design - Fall 2024"
- board text added: "PCB by Jakob Schoeberle"

Commit message: PCB "Done"
Parts:
- J6: footprint Connector_Molex:Molex_Mini-Fit_Jr_5566-24A_2x12_P4.20mm_Vertical -> ThorParts:Molex_Mini-Fit_Jr_5566-24A_2x12_P4.20mm_Vertical_Thor
- moved G*** 108.3 mm to (126.0, 65.5), turned to 0 degrees
- moved J13 8.51 mm to (57.0, 117.0), turned to -90 degrees
- moved J10 8.42 mm to (57.0, 72.2), turned to -90 degrees
- moved J11 8.42 mm to (57.0, 87.2), turned to -90 degrees
- moved J12 8.42 mm to (57.0, 102.2), turned to -90 degrees
- moved REF** 4.47 mm to (163.0, 167.0)
- moved REF** 4.12 mm to (163.0, 134.0)
- moved REF** 3.54 mm to (163.0, 66.0)
- moved REF** 2.92 mm to (57.0, 167.0)
- moved REF** 2.55 mm to (57.0, 66.0)
Connections:
- U7 pad 39: unconnected-(U7-VSYS-Pad39) -> +5V
- U7 pad 40: +5V -> unconnected-(U7-VBUS-Pad40)
Routing:
- net /32A: track 51.3 -> 55.8 mm, vias 0 -> 1
- net /Loadcell_ADCs/-LoadCell3: track 12.2 -> 9.93 mm
- net /Loadcell_ADCs/-LoadCell2: track 12.2 -> 9.88 mm
- net /Loadcell_ADCs/-LoadCell1: track 12.6 -> 10.4 mm
- net /Loadcell_ADCs/-LoadCell4: track 11.5 -> 9.35 mm
- net /13A: track 67.1 -> 65.1 mm
- net Net-(U3-2Y): track 18.4 -> 19.9 mm
- net Net-(U5-2Y): track 18.5 -> 19.9 mm
- net Net-(U4-2Y): track 18.4 -> 19.8 mm
- net Net-(U6-2Y): track 18.4 -> 19.8 mm
- net /Loadcell_ADCs/+LoadCell4: track 10.9 -> 12.2 mm
- net Net-(U4-4Y): track 28.8 -> 30.1 mm
- net /Loadcell_ADCs/+LoadCell3: track 11.6 -> 12.7 mm
- net /Loadcell_ADCs/+LoadCell2: track 11.5 -> 12.6 mm
- net /Loadcell_ADCs/+LoadCell1: track 12.1 -> 13.2 mm
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Other:
- board size 123 x 113.5 mm -> 118 x 112.5 mm
- board text added: "LoadCell_0"
- board text added: "LoadCell_1"
- board text added: "LoadCell_2"
- board text added: "LoadCell_3"
- board text added: "OFF"
- board text added: "ON"
- board text added: "StepperMotor_0"
- board text added: "StepperMotor_1"
- board text added: "StepperMotor_2"
- board text added: "StepperMotor_3"
- board text added: "ThorPCB2.0"
