File: Hardware/ThorPBC2.0.kicad_pcb (KiCad board)
At the start: 4 copper layers, 118 x 112.5 mm, 45 parts, among them J10 LoadCell_0, J11 LoadCell_1, J12 LoadCell_2, J13 LoadCell_3, J5 UART_1, J6 ATX-24, J7 UART_0, J8 ADS1115_Module_1, J9 ADS1115_Module_0, M1 Stepper_Motor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

Commit message: Updates to PCB
Parts:
- moved REF** 2.00 mm to (165.0, 134.0)
- moved REF** 2.00 mm to (165.0, 66.0)
- moved REF** 2.00 mm to (165.0, 167.0)
Routing:
- net /34A: track 30.1 -> 36.3 mm
- net /32A: track 55.8 -> 53.2 mm
- net +5V: track 81.5 -> 83.9 mm
- net /33A: track 45.7 -> 47.4 mm
- net Net-(U5-4Y): track 29.3 -> 29.9 mm
- net /42A: track 72.4 -> 72.9 mm
Other:
- board size 118 x 112.5 mm -> 120 x 112.5 mm

Commit message: Added Back Silkscreen image
Parts:
- added G***: LOGO, ThorParts:CameraMod, B.Cu at (132.1, 137.4)

Commit message: Final Updates
Parts:
- moved G*** 3.97 mm to (129.0, 135.0)
- moved REF** 3.61 mm to (59.0, 69.0)
- moved REF** 3.61 mm to (163.0, 69.0)
- moved REF** 2.83 mm to (59.0, 165.0)
- moved REF** 2.83 mm to (163.0, 165.0)
- moved REF** 2.00 mm to (163.0, 134.0)
- moved C3 1.98 mm to (82.5, 105.6)
- moved C4 1.98 mm to (82.5, 120.7)
- moved J10 1.98 mm to (57.0, 74.2)
- moved J11 1.98 mm to (57.0, 89.2)
- moved J12 1.98 mm to (57.0, 104.2)
- moved J13 1.98 mm to (57.0, 119.0)
- moved R1 1.98 mm to (67.3, 74.8)
- moved R2 1.98 mm to (67.2, 78.9)
- moved R3 1.98 mm to (66.7, 89.8)
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Routing:
- net /Loadcell_ADCs/2_A1: track 17.4 -> 15.4 mm
- net /Loadcell_ADCs/1_A1: track 22.1 -> 20.1 mm
- net /Loadcell_ADCs/1_A2: track 22.1 -> 20.1 mm
- net /Loadcell_ADCs/2_A2: track 17.3 -> 15.5 mm
- net /Loadcell_ADCs/2_A4: track 12.8 -> 14.0 mm
- net /Loadcell_ADCs/2_A3: track 12.7 -> 13.7 mm
- net /Loadcell_ADCs/1_A3: track 14.9 -> 14.1 mm
- net /Loadcell_ADCs/1_A4: track 14.8 -> 14.0 mm
Other:
- board size 120 x 112.5 mm -> 120 x 112 mm
- board text added: "Thoracic Camera Driver Board"
- board text removed: "ThorPCB2.0"
