File: Hardware/ThorPBC2.0.kicad_pcb (KiCad board)
At the start: 4 copper layers, 120 x 112 mm, 46 parts, among them J10 LoadCell_0, J11 LoadCell_1, J12 LoadCell_2, J13 LoadCell_3, J5 UART_1, J6 ATX-24, J7 UART_0, J8 ADS1115_Module_1, J9 ADS1115_Module_0, M1 Stepper_Motor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

Commit message: Updates to PCB
Connections:
- U7 pad 33: unconnected-(U7-AGND-Pad33) -> GND
Changed lines of the file:
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@@
 	(net 68 "/43A")
 	(net 69 "/42A")
-	(net 70 "unconnected-(U7-AGND-Pad33)")
-	(net 71 "unconnected-(U7-GPIO3-Pad5)")
-	(net 72 "unconnected-(U7-VBUS-Pad40)")
-	(net 73 "unconnected-(U7-RUN-Pad30)")
-	(net 74 "unconnected-(U7-GPIO7-Pad10)")
-	(net 75 "unconnected-(U7-GPIO6-Pad9)_0")
-	(net 76 "unconnected-(U7-3V3-Pad36)_0")
-	(net 77 "unconnected-(U7-GND-Pad42)_0")
-	(net 78 "unconnected-(U7-SWCLK-Pad41)")
-	(net 79 "unconnected-(U7-ADC_VREF-Pad35)_0")
-	(net 80 "unconnected-(U7-GPIO2-Pad4)_0")
-	(net 81 "unconnected-(U7-SWDIO-Pad43)_0")
-	(net 82 "unconnected-(U7-3V3_EN-Pad37)_0")
-	(net 83 "unconnected-(U7-GPIO2-Pad4)")
-	(net 84 "unconnected-(U7-ADC_VREF-Pad35)")
-	(net 85 "unconnected-(U7-SWCLK-Pad41)_0")
-	(net 86 "unconnected-(U7-AGND-Pad33)_0")
-	(net 87 "unconnected-(U7-SWDIO-Pad43)")
-	(net 88 "unconnected-(U7-GND-Pad42)")
-	(net 89 "unconnected-(U7-GPIO3-Pad5)_0")
-	(net 90 "unconnected-(U7-3V3-Pad36)")
-	(net 91 "unconnected-(U7-RUN-Pad30)_0")
-	(net 92 "unconnected-(U7-3V3_EN-Pad37)")
-	(net 93 "unconnected-(U7-GPIO6-Pad9)")
-	(net 94 "unconnected-(U7-VBUS-Pad40)_0")
-	(net 95 "unconnected-(U7-GPIO7-Pad10)_0")
+	(net 70 "unconnected-(U7-GPIO3-Pad5)")
+	(net 71 "unconnected-(U7-VBUS-Pad40)")
+	(net 72 "unconnected-(U7-RUN-Pad30)")
+	(net 73 "unconnected-(U7-GPIO7-Pad10)")
+	(net 74 "unconnected-(U7-GPIO6-Pad9)_0")
+	(net 75 "unconnected-(U7-3V3-Pad36)_0")
+	(net 76 "unconnected-(U7-GND-Pad42)_0")
+	(net 77 "unconnected-(U7-SWCLK-Pad41)")
+	(net 78 "unconnected-(U7-ADC_VREF-Pad35)_0")
+	(net 79 "unconnected-(U7-GPIO2-Pad4)_0")
+	(net 80 "unconnected-(U7-SWDIO-Pad43)_0")
+	(net 81 "unconnected-(U7-3V3_EN-Pad37)_0")
+	(net 82 "unconnected-(U7-GPIO2-Pad4)")
+	(net 83 "unconnected-(U7-ADC_VREF-Pad35)")
+	(net 84 "unconnected-(U7-SWCLK-Pad41)_0")
+	(net 85 "unconnected-(U7-SWDIO-Pad43)")
+	(net 86 "unconnected-(U7-GND-Pad42)")
+	(net 87 "unconnected-(U7-GPIO3-Pad5)_0")
+	(net 88 "unconnected-(U7-3V3-Pad36)")
+	(net 89 "unconnected-(U7-RUN-Pad30)_0")
+	(net 90 "unconnected-(U7-3V3_EN-Pad37)")
+	(net 91 "unconnected-(U7-GPIO6-Pad9)")
+	(net 92 "unconnected-(U7-VBUS-Pad40)_0")
+	(net 93 "unconnected-(U7-GPIO7-Pad10)_0")
 	(footprint "ThorParts:CAP_C320_KEM"
 		(layer "F.Cu")
@@
 			)
 		)
+		(property ki_fp_filters "*Mini?Fit*2x12*Vertical* *Mini?Fit*2x12*Horizontal*")
+		(sheetname "Root")
+		(sheetfile "ThorPBC2.0.kicad_sch")
 		(attr through_hole)
 		(fp_line
@@
 			(remove_unused_layers no)
 			(roundrect_rratio 0.09259259259)
-			(net 16 "unconnected-(J6-+3.3V-Pad1)")
+			(net 21 "unconnected-(J6-+3.3V-Pad1)_1")
 			(pinfunction "+3.3V")
 			(pintype "power_out+no_connect")
@@
 			(layers "*.Cu" "*.Mask")
 			(remove_unused_layers no)
-			(net 21 "unconnected-(J6-+3.3V-Pad1)_1")
+			(net 16 "unconnected-(J6-+3.3V-Pad1)")
 			(pinfunction "+3.3V")
 			(pintype "passive+no_connect")
@@
 			)
 		)
-		(fp_text user "${REFERENCE}"
-			(at 0 2 -90)
+		(fp_text user "*"
+			(at -1.7653 0 -90)
 			(unlocked yes)
 			(layer "F.Fab")
@@
 			)
 		)
-		(fp_text user "*"
-			(at -1.7653 0 -90)
+		(fp_text user "${REFERENCE}"
+			(at 0 2 -90)
 			(unlocked yes)
 			(layer "F.Fab")
@@
 			(layers "*.Cu" "*.Mask")
 			(remove_unused_layers no)
-			(net 83 "unconnected-(U7-GPIO2-Pad4)")
+			(net 82 "unconnected-(U7-GPIO2-Pad4)")
 			(pinfunction "GPIO2")
 			(pintype "bidirectional+no_connect")
@@
 			)
 			(layers "F.Cu" "F.Mask")
-			(net 80 "unconnected-(U7-GPIO2-Pad4)_0")
+			(net 79 "unconnected-(U7-GPIO2-Pad4)_0")
 			(pinfunction "GPIO2")
 			(pintype "bidirectional+no_connect")
@@
 			(layers "*.Cu" "*.Mask")
 			(remove_unused_layers no)
-			(net 89 "unconnected-(U7-GPIO3-Pad5)_0")
+			(net 87 "unconnected-(U7-GPIO3-Pad5)_0")
 			(pinfunction "GPIO3")
 			(pintype "bidirectional+no_connect")
@@
 			)
 			(layers "F.Cu" "F.Mask")
-			(net 71 "unconnected-(U7-GPIO3-Pad5)")
+			(net 70 "unconnected-(U7-GPIO3-Pad5)")
 			(pinfunction "GPIO3")
 			(pintype "bidirectional+no_connect")
@@
 			(layers "*.Cu" "*.Mask")
 			(remove_unused_layers no)
-			(net 93 "unconnected-(U7-GPIO6-Pad9)")
+			(net 91 "unconnected-(U7-GPIO6-Pad9)")
 			(pinfunction "GPIO6")
 			(pintype "bidirectional+no_connect")
@@
 			)
 			(layers "F.Cu" "F.Mask")
-			(net 75 "unconnected-(U7-GPIO6-Pad9)_0")
+			(net 74 "unconnected-(U7-GPIO6-Pad9)_0")
 			(pinfunction "GPIO6")
 			(pintype "bidirectional+no_connect")
@@
 			(layers "*.Cu" "*.Mask")
 			(remove_unused_layers no)
-			(net 74 "unconnected-(U7-GPIO7-Pad10)")
+			(net 73 "unconnected-(U7-GPIO7-Pad10)")
 			(pinfunction "GPIO7")
 			(pintype "bidirectional+no_connect")
@@
 			)
 			(layers "F.Cu" "F.Mask")
-			(net 95 "unconnected-(U7-GPIO7-Pad10)_0")
+			(net 93 "unconnected-(U7-GPIO7-Pad10)_0")
 			(pinfunction "GPIO7")
 			(pintype "bidirectional+no_connect")
@@
 			(layers "*.Cu" "*.Mask")
 			(remove_unused_layers no)
-			(net 91 "unconnected-(U7-RUN-Pad30)_0")
+			(net 89 "unconnected-(U7-RUN-Pad30)_0")
 			(pinfunction "RUN")
 			(pintype "input+no_connect")
@@
 			)
 			(layers "F.Cu" "F.Mask")
-			(net 73 "unconnected-(U7-RUN-Pad30)")
+			(net 72 "unconnected-(U7-RUN-Pad30)")
 			(pinfunction "RUN")
 			(pintype "input+no_connect")
@@
 			(layers "*.Cu" "*.Mask")
 			(remove_unused_layers no)
-			(net 86 "unconnected-(U7-AGND-Pad33)_0")
+			(net 10 "GND")
 			(pinfunction "AGND")
-			(pintype "power_in+no_connect")
+			(pintype "power_in")
 		)
 		(pad "33" smd rect
@@
 			)
 			(layers "F.Cu" "F.Mask")
-			(net 70 "unconnected-(U7-AGND-Pad33)")
+			(net 10 "GND")
 			(pinfunction "AGND")
-			(pintype "power_in+no_connect")
+			(pintype "power_in")
 		)
 		(pad "34" thru_hole oval
@@
 			(layers "*.Cu" "*.Mask")
 			(remove_unused_layers no)
-			(net 79 "unconnected-(U7-ADC_VREF-Pad35)_0")
+			(net 78 "unconnected-(U7-ADC_VREF-Pad35)_0")
 			(pinfunction "ADC_VREF")
 			(pintype "power_in+no_connect")
@@
 			)
 			(layers "F.Cu" "F.Mask")
-			(net 84 "unconnected-(U7-ADC_VREF-Pad35)")
+			(net 83 "unconnected-(U7-ADC_VREF-Pad35)")
 			(pinfunction "ADC_VREF")
 			(pintype "power_in+no_connect")
@@
 			(layers "*.Cu" "*.Mask")
 			(remove_unused_layers no)
-			(net 76 "unconnected-(U7-3V3-Pad36)_0")
+			(net 75 "unconnected-(U7-3V3-Pad36)_0")
 			(pinfunction "3V3")
 			(pintype "power_in+no_connect")
@@
 			)
 			(layers "F.Cu" "F.Mask")
-			(net 90 "unconnected-(U7-3V3-Pad36)")
+			(net 88 "unconnected-(U7-3V3-Pad36)")
 			(pinfunction "3V3")
 			(pintype "power_in+no_connect")
@@
 			(layers "*.Cu" "*.Mask")
 			(remove_unused_layers no)
-			(net 82 "unconnected-(U7-3V3_EN-Pad37)_0")
+			(net 81 "unconnected-(U7-3V3_EN-Pad37)_0")
 			(pinfunction "3V3_EN")
 			(pintype "input+no_connect")
@@
 			)
 			(layers "F.Cu" "F.Mask")
-			(net 92 "unconnected-(U7-3V3_EN-Pad37)")
+			(net 90 "unconnected-(U7-3V3_EN-Pad37)")
 			(pinfunction "3V3_EN")
 			(pintype "input+no_connect")
@@
 			(layers "*.Cu" "*.Mask")
 			(remove_unused_layers no)
-			(net 94 "unconnected-(U7-VBUS-Pad40)_0")
+			(net 92 "unconnected-(U7-VBUS-Pad40)_0")
 			(pinfunction "VBUS")
 			(pintype "power_in+no_connect")
@@
 			)
 			(layers "F.Cu" "F.Mask")
-			(net 72 "unconnected-(U7-VBUS-Pad40)")
+			(net 71 "unconnected-(U7-VBUS-Pad40)")
 			(pinfunction "VBUS")
 			(pintype "power_in+no_connect")
@@
 			(layers "*.Cu" "*.Mask")
 			(remove_unused_layers no)
-			(net 85 "unconnected-(U7-SWCLK-Pad41)_0")
+			(net 84 "unconnected-(U7-SWCLK-Pad41)_0")
 			(pinfunction "SWCLK")
 			(pintype "input+no_connect")
@@
 			)
 			(layers "F.Cu" "F.Mask")
-			(net 78 "unconnected-(U7-SWCLK-Pad41)")
+			(net 77 "unconnected-(U7-SWCLK-Pad41)")
 			(pinfunction "SWCLK")
 			(pintype "input+no_connect")
@@
 			(layers "*.Cu" "*.Mask")
 			(remove_unused_layers no)
-			(net 88 "unconnected-(U7-GND-Pad42)")
+			(net 86 "unconnected-(U7-GND-Pad42)")
 			(pinfunction "GND")
 			(pintype "power_in+no_connect")
@@
 			)
 			(layers "F.Cu" "F.Mask")
-			(net 77 "unconnected-(U7-GND-Pad42)_0")
+			(net 76 "unconnected-(U7-GND-Pad42)_0")
 			(pinfunction "GND")
 			(pintype "power_in+no_connect")
@@
 			(layers "*.Cu" "*.Mask")
 			(remove_unused_layers no)
-			(net 81 "unconnected-(U7-SWDIO-Pad43)_0")
+			(net 80 "unconnected-(U7-SWDIO-Pad43)_0")
 			(pinfunction "SWDIO")
 			(pintype "bidirectional+no_connect")
@@
 			)
 			(layers "F.Cu" "F.Mask")
-			(net 87 "unconnected-(U7-SWDIO-Pad43)")
+			(net 85 "unconnected-(U7-SWDIO-Pad43)")
 			(pinfunction "SWDIO")
 			(pintype "bidirectional+no_connect")
@@
 		(polygon
 			(pts
-				(xy 162 113.5) (xy 174 113.5) (xy 174 178) (xy 42.5 178) (xy 42.5 152) (xy 166.5 152) (xy 166.5 121)
-				(xy 162 121)
+				(xy 162 112.5) (xy 174 112.5) (xy 174 178) (xy 42.5 178) (xy 42.5 152) (xy 166.5 152) (xy 166.5 122)
+				(xy 162 122)
 			)
 		)
