File: Hardware/ThorPBC2.0.kicad_sch (KiCad schematic)
At the start: 2 parts, among them J5 Conn_01x03_Pin, J6 ATX-24

Commit message: Updates to PCB
Parts:
- added U7: Pico, MCU_RaspberryPi_and_Boards:RPi_Pico_SMD_TH, symbol MCU_RaspberryPi_and_Boards:Pico
Other:
- company: (none) -> ECE 405 -SIUE
- title: (none) -> ThorPCB2.0
Changed lines of the file:
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@@
 	(generator_version "8.0")
 	(paper "USLetter")
+	(title_block
+		(title "ThorPCB2.0")
+		(company "ECE 405 -SIUE")
+	)
 	(wire
 		(pts
@@
 	(wire
 		(pts
-			(xy 113.03 50.8) (xy 113.03 54.61)
+			(xy 201.93 76.2) (xy 201.93 80.01)
 		)
 		(stroke
@@
 	(wire
 		(pts
-			(xy 106.68 50.8) (xy 113.03 50.8)
+			(xy 195.58 76.2) (xy 201.93 76.2)
 		)
 		(stroke
@@
 	)
 	(symbol
+		(lib_id "MCU_RaspberryPi_and_Boards:Pico")
+		(at 118.11 62.23 0)
+		(unit 1)
+		(exclude_from_sim no)
+		(in_bom yes)
+		(on_board yes)
+		(dnp no)
+		(fields_autoplaced yes)
+		(property "Reference" "U7"
+			(at 118.11 30.48 0)
+			(effects
+				(font
+					(size 1.27 1.27)
+				)
+			)
+		)
+		(property "Value" "Pico"
+			(at 118.11 33.02 0)
+			(effects
+				(font
+					(size 1.27 1.27)
+				)
+			)
+		)
+		(property "Footprint" "MCU_RaspberryPi_and_Boards:RPi_Pico_SMD_TH"
+			(at 118.11 62.23 90)
+			(effects
+				(font
+					(size 1.27 1.27)
+				)
+				(hide yes)
+			)
+		)
+		(property "Datasheet" ""
+			(at 118.11 62.23 0)
+			(effects
+				(font
+					(size 1.27 1.27)
+				)
+				(hide yes)
+			)
+		)
+		(property "Description" ""
+			(at 118.11 62.23 0)
+			(effects
+				(font
+					(size 1.27 1.27)
+				)
+				(hide yes)
+			)
+		)
+		(pin "13"
+		)
+		(pin "8"
+		)
+		(pin "6"
+		)
+		(pin "27"
+		)
+		(pin "42"
+		)
+		(pin "35"
+		)
+		(pin "4"
+		)
+		(pin "17"
+		)
+		(pin "18"
+		)
+		(pin "25"
+		)
+		(pin "12"
+		)
+		(pin "20"
+		)
+		(pin "3"
+		)
+		(pin "32"
+		)
+		(pin "33"
+		)
+		(pin "28"
+		)
+		(pin "41"
+		)
+		(pin "21"
+		)
+		(pin "11"
+		)
+		(pin "26"
+		)
+		(pin "37"
+		)
+		(pin "9"
+		)
+		(pin "31"
+		)
+		(pin "2"
+		)
+		(pin "16"
+		)
+		(pin "30"
+		)
+		(pin "5"
+		)
+		(pin "36"
+		)
+		(pin "29"
+		)
+		(pin "40"
+		)
+		(pin "19"
+		)
+		(pin "38"
+		)
+		(pin "43"
+		)
+		(pin "14"
+		)
+		(pin "15"
+		)
+		(pin "39"
+		)
+		(pin "24"
+		)
+		(pin "7"
+		)
+		(pin "23"
+		)
+		(pin "34"
+		)
+		(pin "22"
+		)
+		(pin "1"
+		)
+		(pin "10"
+		)
+		(instances
+			(project "ThorPBC2.0"
+				(path "/c6e28913-7904-463c-99b0-d22103845470"
+					(reference "U7")
+					(unit 1)
+				)
+			)
+		)
+	)
+	(symbol
 		(lib_id "Connector:ATX-24")
 		(at 35.56 39.37 0)
@@
 	(symbol
 		(lib_id "power:GND")
-		(at 113.03 54.61 0)
+		(at 201.93 80.01 0)
 		(unit 1)
 		(exclude_from_sim no)
@@
 		(dnp no)
 		(property "Reference" "#PWR06"
-			(at 113.03 60.96 0)
+			(at 201.93 86.36 0)
 			(effects
 				(font
@@
 		)
 		(property "Value" "GND"
-			(at 113.03 59.69 0)
+			(at 201.93 85.09 0)
 			(effects
 				(font
@@
 		)
 		(property "Footprint" ""
-			(at 113.03 54.61 0)
+			(at 201.93 80.01 0)
 			(effects
 				(font
@@
 		)
 		(property "Datasheet" ""
-			(at 113.03 54.61 0)
+			(at 201.93 80.01 0)
 			(effects
 				(font
@@
 		)
 		(property "Description" "Power symbol creates a global label with name \"GND\" , ground"
-			(at 113.03 54.61 0)
+			(at 201.93 80.01 0)
 			(effects
 				(font
@@
 	)
 	(sheet
-		(at 87.63 27.94)
+		(at 176.53 53.34)
 		(size 19.05 26.67)
 		(fields_autoplaced yes)
@@
 		)
 		(property "Sheetname" "Loadcell_ADCs"
-			(at 87.63 27.2284 0)
+			(at 176.53 52.6284 0)
 			(effects
 				(font
@@
 		)
 		(property "Sheetfile" "Loadcells_Schematic.kicad_sch"
-			(at 87.63 55.1946 0)
+			(at 176.53 80.5946 0)
 			(effects
 				(font
@@
 		)
 		(pin "VDD" input
-			(at 106.68 31.75 0)
+			(at 195.58 57.15 0)
 			(effects
 				(font
@@
 		)
 		(pin "SCL" bidirectional
-			(at 87.63 31.75 180)
+			(at 176.53 57.15 180)
 			(effects
 				(font
@@
 		)
 		(pin "SDA" bidirectional
-			(at 87.63 36.83 180)
+			(at 176.53 62.23 180)
 			(effects
 				(font
@@
 		)
 		(pin "GND" input
-			(at 106.68 50.8 0)
-			(effects
-				(font
+			(at 195.58 76.2 0)
+			(effects
+				(font

Commit message: Updates to Sch
Parts:
- added J7: Conn_01x03_Pin, symbol Connector:Conn_01x03_Pin
- added SW1: SW_SPDT_321, symbol Switch:SW_SPDT_321
Connections:
- net GND: now also U7.13 (GND), U7.18 (GND), U7.23 (GND), U7.28 (GND), U7.3 (GND), U7.38 (GND), U7.8 (GND), J7.3 (Pin_3), SW1.2 (B)
- net UART_RX: now also U7.12 (GPIO9)
- net UART_TX: now also U7.11 (GPIO8)
- net DEBUG_TX: now reaches U7.1 (GPIO0)
- net DEBUG_TX: now also J7.1 (Pin_1)
- net A1: now reaches U7.14 (GPIO10)
- net A1: now also U7.19 (GPIO14), U7.27 (GPIO21), U7.34 (GPIO28_ADC2)
- net A2: now reaches U7.15 (GPIO11)
- net A2: now also U7.20 (GPIO15), U7.26 (GPIO20), U7.32 (GPIO27_ADC1)
- net A3: now reaches U7.16 (GPIO12)
- net A3: now also U7.22 (GPIO17), U7.25 (GPIO19), U7.31 (GPIO26_ADC0)
- net A4: now reaches U7.17 (GPIO13)
- net A4: now also U7.21 (GPIO16), U7.24 (GPIO18), U7.29 (GPIO22)
- net DEBUG_RX: now reaches U7.2 (GPIO1)
- net DEBUG_RX: now also J7.2 (Pin_2)
- net +5V: now reaches U7.40 (VBUS)
- net +5V: now also J6.21 (+5V), J6.22 (+5V), J6.23 (+5V), J6.4 (+5V), J6.6 (+5V)
- net SDA: now reaches U7.6 (GPIO4)
- net SCL: now reaches U7.7 (GPIO5)
- net +12V: now reaches J6.10 (+12V), J6.11 (+12V)
- net at J6.16 (PS_ON#): now also SW1.3 (A)
- no-connect marks 0 -> 17
Other:
- sheet Loadcell_ADCs ports: added none; removed VDD
- sheet StepperDriver_1 ports: added none; removed VCC1, VCC2
- sheet StepperDriver_2 ports: added none; removed VCC1, VCC2
- sheet StepperDriver_3 ports: added none; removed VCC1, VCC2
- sheet StepperDriver_4 ports: added none; removed VCC1, VCC2
- moved on the sheet: J5, J6, U7

Commit message: PCB Updates
Parts:
- removed SW1: SW_SPDT_321, symbol Switch:SW_SPDT_321
- added SW1: OS102011MS2QN1, SPDT_OS102011_CNK, symbol 2024-10-08_03-09-58:OS102011MS2QN1
- J5, J7: footprint (none) -> Connector_PinHeader_2.54mm:PinHeader_1x03_P2.54mm_Vertical
Connections:
- net GND: now also SW1.2
- net at J6.16 (PS_ON#): now also SW1.1
- removed net A1: U7.14 (GPIO10), U7.19 (GPIO14), U7.27 (GPIO21), U7.34 (GPIO28_ADC2)
- removed net A2: U7.15 (GPIO11), U7.20 (GPIO15), U7.26 (GPIO20), U7.32 (GPIO27_ADC1)
- removed net A3: U7.16 (GPIO12), U7.22 (GPIO17), U7.25 (GPIO19), U7.31 (GPIO26_ADC0)
- removed net A4: U7.17 (GPIO13), U7.21 (GPIO16), U7.24 (GPIO18), U7.29 (GPIO22)
- net DEBUG_RX renamed UART0_RX
- net DEBUG_TX renamed UART0_TX
- net UART_RX renamed UART1_RX
- net UART_TX renamed UART1_TX
- new net 11A: U7.14 (GPIO10)
- new net 12A: U7.15 (GPIO11)
- new net 13A: U7.16 (GPIO12)
- new net 14A: U7.17 (GPIO13)
- new net 21A: U7.19 (GPIO14)
- new net 22A: U7.20 (GPIO15)
- new net 23A: U7.22 (GPIO17)
- new net 24A: U7.21 (GPIO16)
- new net 31A: U7.27 (GPIO21)
- new net 32A: U7.26 (GPIO20)
- new net 33A: U7.25 (GPIO19)
- new net 34A: U7.24 (GPIO18)
- new net 41A: U7.34 (GPIO28_ADC2)
- new net 42A: U7.32 (GPIO27_ADC1)
- new net 43A: U7.31 (GPIO26_ADC0)
- new net 44A: U7.29 (GPIO22)

Commit message: Updates to PCB
Connections:
- no-connect marks 17 -> 18
Changed lines of the file:
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@@
+	)
+	(no_connect
+		(at 30.48 53.34)
 	)
 	(no_connect
@@
 		)
 		(stroke
+			(width 0)
+			(type default)
+		)
+	)
+	(wire
+		(pts
+			(xy 30.48 53.34) (xy 34.29 53.34)
+		)
+		(stroke

Commit message: Updates to PCB
Parts:
- J5: value Conn_01x03_Pin -> UART_1
- J7: value Conn_01x03_Pin -> UART_0
Changed lines of the file:
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@@
 			)
 		)
-		(property "Value" "Conn_01x03_Pin"
+		(property "Value" "UART_0"
 			(at 167.005 71.12 0)
 			(effects
@@
 			)
 		)
-		(property "Value" "Conn_01x03_Pin"
+		(property "Value" "UART_1"
 			(at 167.005 95.25 0)
 			(effects

Commit message: PCB "Done"
Parts:
- J6: footprint Connector_Molex:Molex_Mini-Fit_Jr_5566-24A_2x12_P4.20mm_Vertical -> ThorParts:Molex_Mini-Fit_Jr_5566-24A_2x12_P4.20mm_Vertical_Thor
Connections:
- net +5V: now also U7.39 (VSYS); no longer U7.40 (VBUS)
Changed lines of the file:
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@@
-	)
-	(no_connect
-		(at 114.3 113.03)
 	)
 	(no_connect
@@
 	)
 	(no_connect
+		(at 114.3 110.49)
+	)
+	(no_connect
 		(at 114.3 135.89)
 	)
@@
 		)
 	)
+	(wire
+		(pts
+			(xy 118.11 113.03) (xy 105.41 113.03)
+		)
+		(stroke
+			(width 0)
+			(type default)
+		)
+	)
 	(bus
 		(pts
@@
 	(wire
 		(pts
+			(xy 105.41 110.49) (xy 114.3 110.49)
+		)
+		(stroke
+			(width 0)
+			(type default)
+		)
+	)
+	(wire
+		(pts
 			(xy 64.77 172.72) (xy 110.49 172.72)
 		)
@@
 	(wire
 		(pts
-			(xy 118.11 106.68) (xy 118.11 110.49)
-		)
-		(stroke
-			(width 0)
-			(type default)
-		)
-	)
-	(wire
-		(pts
 			(xy 247.65 120.65) (xy 247.65 124.46)
 		)
@@
 	(wire
 		(pts
+			(xy 118.11 106.68) (xy 118.11 113.03)
+		)
+		(stroke
+			(width 0)
+			(type default)
+		)
+	)
+	(wire
+		(pts
 			(xy 82.55 62.23) (xy 82.55 66.04)
 		)
@@
 	(wire
 		(pts
-			(xy 105.41 110.49) (xy 118.11 110.49)
-		)
-		(stroke
-			(width 0)
-			(type default)
-		)
-	)
-	(wire
-		(pts
 			(xy 30.48 53.34) (xy 34.29 53.34)
 		)
@@
 		(pts
 			(xy 121.92 140.97) (xy 121.92 143.51)
-		)
-		(stroke
-			(width 0)
-			(type default)
-		)
-	)
-	(wire
-		(pts
-			(xy 105.41 113.03) (xy 114.3 113.03)
 		)
 		(stroke
@@
 			)
 		)
-		(property "Footprint" "Connector_Molex:Molex_Mini-Fit_Jr_5566-24A_2x12_P4.20mm_Vertical"
+		(property "Footprint" "ThorParts:Molex_Mini-Fit_Jr_5566-24A_2x12_P4.20mm_Vertical_Thor"
 			(at 82.55 46.99 0)
 			(effects

Commit message: Updates to PCB
Connections:
- net GND: now also U7.33 (AGND)
- no-connect marks 18 -> 17
Changed lines of the file:
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@@
+	)
+	(junction
+		(at 110.49 128.27)
+		(diameter 0)
+		(color 0 0 0 0)
 	)
 	(junction
@@
 	)
 	(no_connect
-		(at 114.3 128.27)
-	)
-	(no_connect
 		(at 30.48 53.34)
 	)
@@
 	(wire
 		(pts
+			(xy 110.49 128.27) (xy 110.49 140.97)
+		)
+		(stroke
+			(width 0)
+			(type default)
+		)
+	)
+	(wire
+		(pts
 			(xy 60.96 130.81) (xy 69.85 130.81)
 		)
@@
 	(wire
 		(pts
-			(xy 105.41 128.27) (xy 114.3 128.27)
-		)
-		(stroke
-			(width 0)
-			(type default)
-		)
-	)
-	(wire
-		(pts
 			(xy 105.41 151.13) (xy 119.38 151.13)
 		)
@@
 	(wire
 		(pts
-			(xy 110.49 115.57) (xy 110.49 140.97)
+			(xy 110.49 115.57) (xy 110.49 128.27)
 		)
 		(stroke
@@
 		)
 		(stroke
+			(width 0)
+			(type default)
+		)
+	)
+	(wire
+		(pts
+			(xy 105.41 128.27) (xy 110.49 128.27)
+		)
+		(stroke
